File: docs/schema/schema.kicad_pcb (KiCad board)
At the start: 2 copper layers, 25 parts, among them J1 IN, J10 Res5, J11 Laser, J12 Capteur porte, J2 Alim driver, J3 Alim Rasberry, J4 Pilotage driver, J5 GPIO Rasberry, J6 Res1, J7 Res2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

Commit message: Update PCB files
Parts:
- added REF**: MountingHole_2.2mm_M2, MountingHole:MountingHole_2.2mm_M2, F.Cu at (124.5, 143.5)
- added REF**: MountingHole_2.2mm_M2, MountingHole:MountingHole_2.2mm_M2, F.Cu at (70.0, 80.5)
- added REF**: MountingHole_2.2mm_M2, MountingHole:MountingHole_2.2mm_M2, F.Cu at (70.0, 143.5)
- added REF**: MountingHole_2.2mm_M2, MountingHole:MountingHole_2.2mm_M2, F.Cu at (124.5, 80.5)
- moved J6 72.7 mm to (81.0, 140.1), turned to 180 degrees
- moved J7 71.3 mm to (87.5, 140.1), turned to 180 degrees
- moved J8 69.9 mm to (94.0, 140.1), turned to 180 degrees
- moved J9 68.6 mm to (100.5, 140.1), turned to 180 degrees
- moved J10 67.3 mm to (107.0, 140.1), turned to 180 degrees
- moved J5 66.6 mm to (74.5, 100.5)
- moved R4 66.6 mm to (100.9, 115.0)
- moved R3 65.6 mm to (99.4, 109.0)
- moved R2 64.7 mm to (98.0, 103.0)
- moved R1 64.0 mm to (96.4, 97.0)
- moved J3 57.3 mm to (74.5, 87.0)
- moved R8 56.9 mm to (99.4, 112.5), turned to 0 degrees
- moved R7 56.5 mm to (97.9, 106.5), turned to 0 degrees
- moved R5 56.3 mm to (94.9, 94.5), turned to 0 degrees
- moved R6 56.3 mm to (96.5, 100.5), turned to 0 degrees
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Connections:
- J11 pad 1: GND -> Net-(J11-Pin_1)
- J11 pad 2: Net-(J11-Pin_2) -> +5V
- J12 pad 1: GND -> Net-(J12-Pin_1)
- J12 pad 2: Net-(J12-Pin_2) -> +3.3V
- J5 pad 5: Net-(J12-Pin_2) -> Net-(J12-Pin_1)
- Q1 pad 3: Net-(J11-Pin_2) -> Net-(J11-Pin_1)
Routing:
- net +5V: track 0.00 -> 155.6 mm
- net +3.3V: track 0.00 -> 96.5 mm
- net Net-(J12-Pin_1): track 0.00 -> 56.1 mm
- net Net-(J10-Pin_4): track 0.00 -> 40.5 mm
- net +24V: track 0.00 -> 34.8 mm
- net Net-(J5-Pin_7): track 0.00 -> 32.9 mm
- net Net-(J11-Pin_1): track 0.00 -> 27.7 mm
- net Net-(J4-Pin_4): track 0.00 -> 26.9 mm
- net Net-(J5-Pin_8): track 0.00 -> 25.4 mm
- net Net-(J5-Pin_4): track 0.00 -> 25.3 mm
- net Net-(J4-Pin_3): track 0.00 -> 24.1 mm
- net Net-(J5-Pin_3): track 0.00 -> 22.3 mm
- net Net-(J4-Pin_1): track 0.00 -> 22.2 mm
- net Net-(J5-Pin_2): track 0.00 -> 21.6 mm
- net Net-(J5-Pin_1): track 0.00 -> 21.4 mm
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- added copper zone on B.Cu, net GND
Other:
- board outline added: 59.5 x 68 mm
