File: docs/schema/schema.kicad_sch (KiCad schematic)
At the start: 2 parts, among them U1 24V1, U2 24V2

Commit message: WIP: Schema
Parts:
- removed U1: 24V1, Library_Perso:Connector_boxed_2.54_1x02, symbol Library_Perso:connector_boxed_2.54mm_1x02
- removed U2: 24V2, Library_Perso:Connector_boxed_2.54_1x02, symbol Library_Perso:connector_boxed_2.54mm_1x02
- added J1: IN, Connector_JST:JST_PH_B2B-PH-K_1x02_P2.00mm_Vertical, symbol Connector:Conn_01x02_Pin
- added J10: Res5, Connector_JST:JST_PH_B4B-PH-K_1x04_P2.00mm_Vertical, symbol Connector:Conn_01x04_Pin
- added J11: Laser, Connector_JST:JST_PH_B2B-PH-K_1x02_P2.00mm_Vertical, symbol Connector:Conn_01x02_Pin
- added J12: Capteur porte, Connector_JST:JST_PH_B2B-PH-K_1x02_P2.00mm_Vertical, symbol Connector:Conn_01x02_Pin
- added J2: Alim driver, Connector_JST:JST_PH_B2B-PH-K_1x02_P2.00mm_Vertical, symbol Connector:Conn_01x02_Pin
- added J3: Alim Rasberry, Connector_JST:JST_PH_B3B-PH-K_1x03_P2.00mm_Vertical, symbol Connector:Conn_01x03_Pin
- added J4: Pilotage driver, Connector_JST:JST_PH_B4B-PH-K_1x04_P2.00mm_Vertical, symbol Connector:Conn_01x04_Pin
- added J5: GPIO Rasberry, Connector_JST:JST_PH_B10B-PH-K_1x10_P2.00mm_Vertical, symbol Connector:Conn_01x10_Pin
- added J6: Res1, Connector_JST:JST_PH_B4B-PH-K_1x04_P2.00mm_Vertical, symbol Connector:Conn_01x04_Pin
- added J7: Res2, Connector_JST:JST_PH_B4B-PH-K_1x04_P2.00mm_Vertical, symbol Connector:Conn_01x04_Pin
- added J8: Res3, Connector_JST:JST_PH_B4B-PH-K_1x04_P2.00mm_Vertical, symbol Connector:Conn_01x04_Pin
- added J9: Res4, Connector_JST:JST_PH_B4B-PH-K_1x04_P2.00mm_Vertical, symbol Connector:Conn_01x04_Pin
- added Q1, Q2, Q3, Q4: Q_NMOS_DGS, symbol Transistor_FET:Q_NMOS_DGS
- added R1, R2, R3, R4: R, symbol Device:R
Connections:
- net +24V: now also J1.2 (Pin_2), J2.2 (Pin_2)
- net GND: now also J1.1 (Pin_1), J10.3 (Pin_3), J12.1 (Pin_1), J2.1 (Pin_1), J3.1 (Pin_1), J6.3 (Pin_3), J7.3 (Pin_3), J8.3 (Pin_3), J9.3 (Pin_3), Q1.3 (S), Q2.3 (S), Q3.3 (S), Q4.3 (S), R1.2, R2.2, R3.2, R4.2
- new net: J5.1 (Pin_1), Q1.2 (G), R1.1
- new net: J5.10 (Pin_10), J6.4 (Pin_4)
- new net: J5.2 (Pin_2), Q2.2 (G), R2.1
- new net: J5.3 (Pin_3), Q3.2 (G), R3.1
- new net: J5.4 (Pin_4), Q4.2 (G), R4.1
- new net: J12.2 (Pin_2), J5.5 (Pin_5)
- new net: J10.4 (Pin_4), J5.6 (Pin_6)
- new net: J5.7 (Pin_7), J9.4 (Pin_4)
- new net: J5.8 (Pin_8), J8.4 (Pin_4)
- new net: J5.9 (Pin_9), J7.4 (Pin_4)
- new net +3.3V: J10.2 (Pin_2), J3.2 (Pin_2), J6.2 (Pin_2), J7.2 (Pin_2), J8.2 (Pin_2), J9.2 (Pin_2)
- new net +5V: J10.1 (Pin_1), J3.3 (Pin_3), J6.1 (Pin_1), J7.1 (Pin_1), J8.1 (Pin_1), J9.1 (Pin_1)

Commit message: Draw PCB schematic
Parts:
- removed Q1, Q2, Q3, Q4: Q_NMOS_DGS, symbol Transistor_FET:Q_NMOS_DGS
- added Q1, Q2, Q3, Q4: SI2302, Package_TO_SOT_SMD:SOT-23, symbol Transistor_FET:AO3400A
- added R5, R6, R7, R8: 100, Resistor_SMD:R_1206_3216Metric, symbol Device:R
- added U1: LM2596, Library_Perso:LM2596 module, symbol Library_Perso:LM2596_module
- J1, J11, J12, J2: footprint Connector_JST:JST_PH_B2B-PH-K_1x02_P2.00mm_Vertical -> Connector_PinHeader_2.54mm:PinHeader_1x02_P2.54mm_Vertical
- J10, J4, J6, J7, J8, J9: footprint Connector_JST:JST_PH_B4B-PH-K_1x04_P2.00mm_Vertical -> Connector_PinHeader_2.54mm:PinHeader_1x04_P2.54mm_Vertical
- J3: footprint Connector_JST:JST_PH_B3B-PH-K_1x03_P2.00mm_Vertical -> Connector_PinHeader_2.54mm:PinHeader_1x03_P2.54mm_Vertical
- J5: footprint Connector_JST:JST_PH_B10B-PH-K_1x10_P2.00mm_Vertical -> Connector_PinHeader_2.54mm:PinHeader_1x10_P2.54mm_Vertical
- R1, R2, R3, R4: value R -> 100k; footprint (none) -> Resistor_SMD:R_1206_3216Metric
Connections:
- net +24V: now also U1.IN+
- net +5V: now also J4.2 (Pin_2), U1.OUT+
- net GND: now also J11.1 (Pin_1), Q1.2 (S), Q2.2 (S), Q3.2 (S), Q4.2 (S), U1.IN-, U1.OUT-
- net at J5.1 (Pin_1): now also R5.1; no longer R1.1
- net at J5.2 (Pin_2): now also R6.1; no longer R2.1
- net at J5.3 (Pin_3): now also R7.1; no longer R3.1
- net at J5.4 (Pin_4): now also R8.1; no longer R4.1
- net at J4.1 (Pin_1): now also Q4.3 (D)
- net at J4.3 (Pin_3): now also Q3.3 (D)
- net at J4.4 (Pin_4): now also Q2.3 (D)
- net at J11.2 (Pin_2): now also Q1.3 (D)
- new net: Q4.1 (G), R4.1, R8.2
- new net: Q1.1 (G), R1.1, R5.2
- new net: Q3.1 (G), R3.1, R7.2
- new net: Q2.1 (G), R2.1, R6.2
Other:
- moved on the sheet: J1, J10, J11, J12, J2, J3, J4, J5, J6, J7, J8, J9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

Commit message: Update PCB files
Connections:
- net +3.3V: now also J12.2 (Pin_2)
- net +5V: now also J11.2 (Pin_2)
- net GND: no longer J11.1 (Pin_1), J12.1 (Pin_1)
- net at J5.5 (Pin_5): now also J12.1 (Pin_1); no longer J12.2 (Pin_2)
- net at Q1.3 (D): now also J11.1 (Pin_1); no longer J11.2 (Pin_2)
Changed lines of the file:
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@@
+	(wire
+		(pts
+			(xy 111.76 135.89) (xy 111.76 134.62)
+		)
+		(stroke
+			(width 0)
+			(type default)
+		)
+	)
 	(wire
 		(pts
@@
 	(wire
 		(pts
-			(xy 113.03 135.89) (xy 58.42 135.89)
-		)
-		(stroke
-			(width 0)
-			(type default)
-		)
-	)
-	(wire
-		(pts
 			(xy 63.5 118.11) (xy 68.58 118.11)
 		)
@@
 	(wire
 		(pts
-			(xy 58.42 101.6) (xy 58.42 135.89)
-		)
-		(stroke
-			(width 0)
-			(type default)
-		)
-	)
-	(wire
-		(pts
 			(xy 58.42 101.6) (xy 43.18 101.6)
 		)
@@
 	(wire
 		(pts
+			(xy 113.03 138.43) (xy 58.42 138.43)
+		)
+		(stroke
+			(width 0)
+			(type default)
+		)
+	)
+	(wire
+		(pts
 			(xy 53.34 104.14) (xy 53.34 149.86)
 		)
@@
 	(wire
 		(pts
+			(xy 113.03 63.5) (xy 111.76 63.5)
+		)
+		(stroke
+			(width 0)
+			(type default)
+		)
+	)
+	(wire
+		(pts
 			(xy 63.5 91.44) (xy 63.5 72.39)
 		)
@@
 	(wire
 		(pts
+			(xy 111.76 63.5) (xy 111.76 62.23)
+		)
+		(stroke
+			(width 0)
+			(type default)
+		)
+	)
+	(wire
+		(pts
 			(xy 100.33 39.37) (xy 100.33 40.64)
 		)
@@
 	(wire
 		(pts
-			(xy 85.09 63.5) (xy 113.03 63.5)
-		)
-		(stroke
-			(width 0)
-			(type default)
-		)
-	)
-	(wire
-		(pts
 			(xy 69.85 157.48) (xy 69.85 166.37)
 		)
@@
 	(wire
 		(pts
-			(xy 85.09 67.31) (xy 85.09 63.5)
+			(xy 113.03 135.89) (xy 111.76 135.89)
+		)
+		(stroke
+			(width 0)
+			(type default)
+		)
+	)
+	(wire
+		(pts
+			(xy 85.09 67.31) (xy 85.09 66.04)
 		)
 		(stroke
@@
 	(wire
 		(pts
+			(xy 85.09 66.04) (xy 113.03 66.04)
+		)
+		(stroke
+			(width 0)
+			(type default)
+		)
+	)
+	(wire
+		(pts
 			(xy 66.04 102.87) (xy 68.58 102.87)
 		)
@@
 		(pts
 			(xy 43.18 104.14) (xy 53.34 104.14)
+		)
+		(stroke
+			(width 0)
+			(type default)
+		)
+	)
+	(wire
+		(pts
+			(xy 58.42 101.6) (xy 58.42 138.43)
 		)
 		(stroke
@@
 	)
 	(symbol
-		(lib_id "power:GND")
-		(at 113.03 66.04 0)
+		(lib_id "power:+5V")
+		(at 111.76 62.23 0)
 		(unit 1)
 		(body_style 1)
@@
 		(fields_autoplaced yes)
 		(property "Reference" "#PWR019"
-			(at 113.03 72.39 0)
-			(hide yes)
-			(show_name no)
-			(do_not_autoplace no)
-			(effects
-				(font
-					(size 1.27 1.27)
-				)
-			)
-		)
-		(property "Value" "GND"
-			(at 113.03 71.12 0)
+			(at 111.76 66.04 0)
+			(hide yes)
+			(show_name no)
+			(do_not_autoplace no)
+			(effects
+				(font
+					(size 1.27 1.27)
+				)
+			)
+		)
+		(property "Value" "+5V"
+			(at 111.76 57.15 0)
 			(show_name no)
 			(do_not_autoplace no)
@@
 		)
 		(property "Footprint" ""
-			(at 113.03 66.04 0)
+			(at 111.76 62.23 0)
 			(hide yes)
 			(show_name no)
@@
 		)
 		(property "Datasheet" ""
-			(at 113.03 66.04 0)
-			(hide yes)
-			(show_name no)
-			(do_not_autoplace no)
-			(effects
-				(font
-					(size 1.27 1.27)
-				)
-			)
-		)
-		(property "Description" "Power symbol creates a global label with name \"GND\" , ground"
-			(at 113.03 66.04 0)
+			(at 111.76 62.23 0)
+			(hide yes)
+			(show_name no)
+			(do_not_autoplace no)
+			(effects
+				(font
+					(size 1.27 1.27)
+				)
+			)
+		)
+		(property "Description" "Power symbol creates a global label with name \"+5V\""
+			(at 111.76 62.23 0)
 			(hide yes)
 			(show_name no)
@@
 	)
 	(symbol
+		(lib_id "power:+3.3V")
+		(at 111.76 134.62 0)
+		(unit 1)
+		(body_style 1)
+		(exclude_from_sim no)
+		(in_bom yes)
+		(on_board yes)
+		(in_pos_files yes)
+		(dnp no)
+		(fields_autoplaced yes)
+		(property "Reference" "#PWR015"
+			(at 111.76 138.43 0)
+			(hide yes)
+			(show_name no)
+			(do_not_autoplace no)
+			(effects
+				(font
+					(size 1.27 1.27)
+				)
+			)
+		)
+		(property "Value" "+3.3V"
+			(at 111.76 129.54 0)
+			(show_name no)
+			(do_not_autoplace no)
+			(effects
+				(font
+					(size 1.27 1.27)
+				)
+			)
+		)
+		(property "Footprint" ""
+			(at 111.76 134.62 0)
+			(hide yes)
+			(show_name no)
+			(do_not_autoplace no)
+			(effects
+				(font
+					(size 1.27 1.27)
+				)
+			)
+		)
+		(property "Datasheet" ""
+			(at 111.76 134.62 0)
+			(hide yes)
+			(show_name no)
+			(do_not_autoplace no)
+			(effects
+				(font
+					(size 1.27 1.27)
+				)
+			)
+		)
+		(property "Description" "Power symbol creates a global label with name \"+3.3V\""
+			(at 111.76 134.62 0)
+			(hide yes)
+			(show_name no)
+			(do_not_autoplace no)
+			(effects
+				(font
+					(size 1.27 1.27)
+				)
+			)
+		)
+		(pin "1"
+		)
+		(instances
+			(project "schema"
+				(path "/b5f0736d-188b-4a2a-9d72-b6406c626165"
+					(reference "#PWR015")
+					(unit 1)
+				)
+			)
+		)
+	)
+	(symbol
 		(lib_id "Device:R")
 		(at 77.47 91.44 0)
@@
 					(unit 1)
 				)
-			)
-		)
-	)
-	(symbol
-		(lib_id "power:GND")
-		(at 113.03 138.43 0)
-		(unit 1)
-		(body_style 1)
-		(exclude_from_sim no)
-		(in_bom yes)
-		(on_board yes)
-		(in_pos_files yes)
-		(dnp no)
-		(fields_autoplaced yes)
-		(property "Reference" "#PWR015"
-			(at 113.03 144.78 0)
-			(hide yes)
-			(show_name no)
-			(do_not_autoplace no)
-			(effects
-				(font
-					(size 1.27 1.27)
-				)
-			)
-		)
-		(property "Value" "GND"
-			(at 113.03 143.51 0)
-			(show_name no)
-			(do_not_autoplace no)
-			(effects
-				(font
-					(size 1.27 1.27)
-				)
-			)
-		)
-		(property "Footprint" ""
-			(at 113.03 138.43 0)
-			(hide yes)
-			(show_name no)
-			(do_not_autoplace no)
-			(effects
-				(font
-					(size 1.27 1.27)
-				)
-			)
-		)
-		(property "Datasheet" ""
-			(at 113.03 138.43 0)
-			(hide yes)
-			(show_name no)
-			(do_not_autoplace no)
-			(effects
-				(font
-					(size 1.27 1.27)
-				)
-			)
-		)
-		(property "Description" "Power symbol creates a global label with name \"GND\" , ground"
-			(at 113.03 138.43 0)
-			(hide yes)
-			(show_name no)
-			(do_not_autoplace no)
-			(effects
-				(font
-					(size 1.27 1.27)
-				)
-			)
-		)
-		(pin "1"
-		)
-		(instances
-			(project "schema"
-				(path "/b5f0736d-188b-4a2a-9d72-b6406c626165"
-					(reference "#PWR015")
-					(unit 1)
-				)
